File: HAM_Seminiar_Opamp/HAM_Seminiar_Opamp/HAM_Seminiar_Opamp.kicad_pcb (KiCad board)
At the start: 2 copper layers, 104 x 72 mm, 24 parts, among them J1 Conn_01x02_Pin, SW1 SW_SPDT, U1 LM741, U2 LM1117MP-1.8, U3 LM311, U4 LM311, U5 LM311, U6 LM311

Commit message: s
Other:
- board size 104 x 72 mm -> 99.9 x 69.5 mm
Changed lines of the file:
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@@
 			(outputformat 1)
 			(mirror no)
-			(drillshape 1)
+			(drillshape 0)
 			(scaleselection 1)
-			(outputdirectory "")
+			(outputdirectory "gerber")
 		)
 	)
@@
 	)
 	(gr_rect
-		(start 68 65)
-		(end 172 137)
+		(start 70.54 65)
+		(end 170.476 134.46)
 		(stroke
 			(width 0.05)
