File: HAM_Seminar/HAM_Seminar.kicad_sch (KiCad schematic)
At the start: 17 parts, among them J2 Conn_01x02_Socket, U1 NE555P, U2 74LS90, U3 74LS48, U4 MAN3840A

Commit message: sERT
Parts:
- removed J2: Conn_01x02_Socket, Connector_PinHeader_2.54mm:PinHeader_1x02_P2.54mm_Vertical, symbol Connector:Conn_01x02_Socket
- removed U4: MAN3840A, Display_7Segment:MAN3810A, symbol Display_Character:MAN3840A
- added BT1: Battery, Connector_PinHeader_2.54mm:PinHeader_1x02_P2.54mm_Vertical, symbol Device:Battery
- added SW1: SW_SPDT, Connector_Molex:Molex_Micro-Fit_3.0_43650-0315_1x03_P3.00mm_Vertical, symbol Switch:SW_SPDT
- added U4: D148K, Display_7Segment:D1X8K, symbol Display_Character:D148K
- C1: footprint Capacitor_THT:C_Radial_D4.0mm_H7.0mm_P1.50mm -> Capacitor_THT:C_Radial_D5.0mm_H5.0mm_P2.00mm
- C2: footprint Capacitor_THT:C_Radial_D4.0mm_H7.0mm_P1.50mm -> Capacitor_THT:C_Disc_D4.3mm_W1.9mm_P5.00mm
- R1: renamed from R2; footprint Resistor_THT:R_Axial_DIN0207_L6.3mm_D2.5mm_P10.16mm_Horizontal -> Resistor_THT:R_Axial_DIN0204_L3.6mm_D1.6mm_P7.62mm_Horizontal
- R10: renamed from R9; footprint Resistor_THT:R_Axial_DIN0207_L6.3mm_D2.5mm_P10.16mm_Horizontal -> Resistor_THT:R_Axial_DIN0204_L3.6mm_D1.6mm_P7.62mm_Horizontal
- R2: renamed from R10; footprint Resistor_THT:R_Axial_DIN0207_L6.3mm_D2.5mm_P10.16mm_Horizontal -> Resistor_THT:R_Axial_DIN0204_L3.6mm_D1.6mm_P7.62mm_Horizontal
- R3: renamed from R1; footprint Resistor_THT:R_Axial_DIN0207_L6.3mm_D2.5mm_P10.16mm_Horizontal -> Resistor_THT:R_Axial_DIN0204_L3.6mm_D1.6mm_P7.62mm_Horizontal
- R4: renamed from R3; footprint Resistor_THT:R_Axial_DIN0207_L6.3mm_D2.5mm_P10.16mm_Horizontal -> Resistor_THT:R_Axial_DIN0204_L3.6mm_D1.6mm_P7.62mm_Horizontal
- R5: renamed from R4; footprint Resistor_THT:R_Axial_DIN0207_L6.3mm_D2.5mm_P10.16mm_Horizontal -> Resistor_THT:R_Axial_DIN0204_L3.6mm_D1.6mm_P7.62mm_Horizontal
- R6: renamed from R5; footprint Resistor_THT:R_Axial_DIN0207_L6.3mm_D2.5mm_P10.16mm_Horizontal -> Resistor_THT:R_Axial_DIN0204_L3.6mm_D1.6mm_P7.62mm_Horizontal
- R7: renamed from R6; footprint Resistor_THT:R_Axial_DIN0207_L6.3mm_D2.5mm_P10.16mm_Horizontal -> Resistor_THT:R_Axial_DIN0204_L3.6mm_D1.6mm_P7.62mm_Horizontal
- R8: renamed from R7; footprint Resistor_THT:R_Axial_DIN0207_L6.3mm_D2.5mm_P10.16mm_Horizontal -> Resistor_THT:R_Axial_DIN0204_L3.6mm_D1.6mm_P7.62mm_Horizontal
- R9: renamed from R8; footprint Resistor_THT:R_Axial_DIN0207_L6.3mm_D2.5mm_P10.16mm_Horizontal -> Resistor_THT:R_Axial_DIN0204_L3.6mm_D1.6mm_P7.62mm_Horizontal
- U2: footprint Package_DIP:DIP-12_W7.62mm -> Package_DIP:DIP-14_W7.62mm
Connections:
- net GND: now also BT1.2 (-), U4.3 (CC), U4.8 (CC)
- net VCC: now also SW1.1 (A)
- net at R3.2: now also U4.7 (A)
- net at R4.2: now also U4.6 (B)
- net at R10.2: now also U4.5 (DP)
- net at R8.2: now also U4.9 (F)
- net at R9.2: now also U4.10 (G)
- net at R7.2: now also U4.1 (E)
- net at R6.2: now also U4.2 (D)
- net at R5.2: now also U4.4 (C)
- new net: BT1.1 (+), SW1.2 (B)
Other:
- note added: "NE555 발진 회로 - 1kHz R1 = 5kΩ, R2 = 4.7kΩ, C = 100nF f = 1.44/((5k+2×4.7k)×100n) = 1kHz duty = (5k+4.7k)/(5k+2×4.7k) = 67%"
- note added: "VCC = 5V 입력 터미널"
- note removed: "R1 = 10k R2 = 0k~10k f = 1.44/(2~12)*1u = 72Hz ~ 48Hz = 1440/(20~30) duty = 0.5~0.7 = 1- (0~10)/(10k~30k)"
- note removed: "R1 = 10k R2 = 10k C = 100u f = 1.44/((30k)*100u) = 0.48Hz duty = 1- (10)/(30k) = 0.7"
- note removed: "T=0.693(R1+R2)C1 f=1.44/(R1+2R2)C1 duty = (R1+R2)/(R1+2R2) = 1-R2/(R1+2R2)"

Commit message: final
Parts:
- C1: value 100u -> 10u
- C2: value C -> 100nF
- R1, R10, R2, R4, R5, R6, R7, R8, R9: footprint Resistor_THT:R_Axial_DIN0204_L3.6mm_D1.6mm_P7.62mm_Horizontal -> Resistor_THT:R_Axial_DIN0207_L6.3mm_D2.5mm_P10.16mm_Horizontal
- R3: value R -> 100R; footprint Resistor_THT:R_Axial_DIN0204_L3.6mm_D1.6mm_P7.62mm_Horizontal -> Resistor_THT:R_Axial_DIN0207_L6.3mm_D2.5mm_P10.16mm_Horizontal
- U3: value 74LS48 -> 74LS47
- U4: value D148K -> D148A
Connections:
- net GND: no longer U4.3 (CC), U4.8 (CC)
- net VCC: now also U4.3 (CC), U4.8 (CC)
Changed lines of the file:
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@@
 	(text "NE555 발진 회로 - 1kHz\nR1 = 5kΩ, R2 = 4.7kΩ, C = 100nF\nf = 1.44/((5k+2×4.7k)×100n) = 1kHz\nduty = (5k+4.7k)/(5k+2×4.7k) = 67%\n"
 		(exclude_from_sim no)
-		(at 50 50 0)
+		(at 49.53 39.878 0)
 		(effects
 			(font
@@
 	)
 	(junction
+		(at 247.65 100.33)
+		(diameter 0)
+		(color 0 0 0 0)
+	)
+	(junction
 		(at 148.59 102.87)
 		(diameter 0)
@@
 	)
 	(junction
-		(at 247.65 102.87)
-		(diameter 0)
-		(color 0 0 0 0)
-	)
-	(junction
 		(at 180.34 85.09)
 		(diameter 0)
@@
 	(wire
 		(pts
-			(xy 247.65 102.87) (xy 247.65 114.3)
-		)
-		(stroke
-			(width 0)
-			(type default)
-		)
-	)
-	(wire
-		(pts
 			(xy 229.87 85.09) (xy 224.79 85.09)
 		)
@@
 		(pts
 			(xy 217.17 85.09) (xy 212.09 85.09)
+		)
+		(stroke
+			(width 0)
+			(type default)
+		)
+	)
+	(wire
+		(pts
+			(xy 247.65 69.85) (xy 247.65 100.33)
 		)
 		(stroke
@@
 		(on_board yes)
 		(dnp no)
-		(fields_autoplaced yes)
 		(property "Reference" "R3"
-			(at 220.98 78.74 90)
-			(effects
-				(font
-					(size 1.27 1.27)
-				)
-			)
-		)
-		(property "Value" "R"
-			(at 220.98 81.28 90)
-			(effects
-				(font
-					(size 1.27 1.27)
-				)
-			)
-		)
-		(property "Footprint" "Resistor_THT:R_Axial_DIN0204_L3.6mm_D1.6mm_P7.62mm_Horizontal"
+			(at 219.71 66.802 90)
+			(effects
+				(font
+					(size 1.27 1.27)
+				)
+			)
+		)
+		(property "Value" "100R"
+			(at 225.552 81.28 90)
+			(effects
+				(font
+					(size 1.27 1.27)
+				)
+			)
+		)
+		(property "Footprint" "Resistor_THT:R_Axial_DIN0207_L6.3mm_D2.5mm_P10.16mm_Horizontal"
 			(at 220.98 86.868 90)
 			(effects
@@
 			)
 		)
-		(property "Value" "74LS48"
+		(property "Value" "74LS47"
 			(at 201.5333 80.01 0)
 			(effects
@@
 		(on_board yes)
 		(dnp no)
-		(fields_autoplaced yes)
 		(property "Reference" "R4"
-			(at 220.98 81.28 90)
+			(at 219.71 68.834 90)
 			(effects
 				(font
@@
 		)
 		(property "Value" "R"
-			(at 220.98 83.82 90)
-			(effects
-				(font
-					(size 1.27 1.27)
-				)
-			)
-		)
-		(property "Footprint" "Resistor_THT:R_Axial_DIN0204_L3.6mm_D1.6mm_P7.62mm_Horizontal"
+			(at 224.028 80.772 90)
+			(effects
+				(font
+					(size 1.27 1.27)
+				)
+				(hide yes)
+			)
+		)
+		(property "Footprint" "Resistor_THT:R_Axial_DIN0207_L6.3mm_D2.5mm_P10.16mm_Horizontal"
 			(at 220.98 89.408 90)
 			(effects
@@
 		(on_board yes)
 		(dnp no)
-		(fields_autoplaced yes)
 		(property "Reference" "R10"
-			(at 220.98 99.06 90)
+			(at 220.218 81.28 90)
 			(effects
 				(font
@@
 					(size 1.27 1.27)
 				)
-			)
-		)
-		(property "Footprint" "Resistor_THT:R_Axial_DIN0204_L3.6mm_D1.6mm_P7.62mm_Horizontal"
+				(hide yes)
+			)
+		)
+		(property "Footprint" "Resistor_THT:R_Axial_DIN0207_L6.3mm_D2.5mm_P10.16mm_Horizontal"
 			(at 220.98 107.188 90)
 			(effects
@@
 			)
 		)
-		(property "Value" "D148K"
+		(property "Value" "D148A"
 			(at 237.49 77.47 0)
 			(effects
@@
 		(lib_id "Device:C")
 		(at 114.3 107.95 0)
-		(unit 1)
-		(exclude_from_sim no)
-		(in_bom yes)
-		(on_board yes)
-		(dnp no)
-		(fields_autoplaced yes)
+		(mirror y)
+		(unit 1)
+		(exclude_from_sim no)
+		(in_bom yes)
+		(on_board yes)
+		(dnp no)
 		(property "Reference" "C2"
-			(at 118.11 106.6799 0)
+			(at 110.49 106.6799 0)
 			(effects
 				(font
@@
 			)
 		)
-		(property "Value" "C"
-			(at 118.11 109.2199 0)
+		(property "Value" "100nF"
+			(at 110.49 109.2199 0)
 			(effects
 				(font
@@
 		)
 		(property "Footprint" "Capacitor_THT:C_Disc_D4.3mm_W1.9mm_P5.00mm"
-			(at 115.2652 111.76 0)
+			(at 113.3348 111.76 0)
 			(effects
 				(font
@@
 			)
 		)
-		(property "Value" "100u"
+		(property "Value" "10u"
 			(at 96.52 109.2199 0)
 			(effects
@@
 			)
 		)
-		(property "Footprint" "Resistor_THT:R_Axial_DIN0204_L3.6mm_D1.6mm_P7.62mm_Horizontal"
+		(property "Footprint" "Resistor_THT:R_Axial_DIN0207_L6.3mm_D2.5mm_P10.16mm_Horizontal"
 			(at 90.932 77.47 90)
 			(effects
@@
 		(on_board yes)
 		(dnp no)
-		(fields_autoplaced yes)
 		(property "Reference" "R5"
-			(at 220.98 83.82 90)
+			(at 219.71 70.866 90)
 			(effects
 				(font
@@
 					(size 1.27 1.27)
 				)
-			)
-		)
-		(property "Footprint" "Resistor_THT:R_Axial_DIN0204_L3.6mm_D1.6mm_P7.62mm_Horizontal"
+				(hide yes)
+			)
+		)
+		(property "Footprint" "Resistor_THT:R_Axial_DIN0207_L6.3mm_D2.5mm_P10.16mm_Horizontal"
 			(at 220.98 91.948 90)
 			(effects
@@
 		(on_board yes)
 		(dnp no)
-		(fields_autoplaced yes)
 		(property "Reference" "R7"
-			(at 220.98 88.9 90)
+			(at 219.71 74.93 90)
 			(effects
 				(font
@@
 					(size 1.27 1.27)
 				)
-			)
-		)
-		(property "Footprint" "Resistor_THT:R_Axial_DIN0204_L3.6mm_D1.6mm_P7.62mm_Horizontal"
+				(hide yes)
+			)
+		)
+		(property "Footprint" "Resistor_THT:R_Axial_DIN0207_L6.3mm_D2.5mm_P10.16mm_Horizontal"
 			(at 220.98 97.028 90)
 			(effects
@@
 				(path "/7b2739d8-9b30-4e41-8527-a1823fcf2f65"
 					(reference "R7")
+					(unit 1)
+				)
+			)
+		)
+	)
+	(symbol
+		(lib_id "power:VCC")
+		(at 247.65 69.85 0)
+		(unit 1)
+		(exclude_from_sim no)
+		(in_bom yes)
+		(on_board yes)
+		(dnp no)
+		(fields_autoplaced yes)
+		(property "Reference" "#PWR015"
+			(at 247.65 73.66 0)
+			(effects
+				(font
+					(size 1.27 1.27)
+				)
+				(hide yes)
+			)
+		)
+		(property "Value" "VCC"
+			(at 247.65 64.77 0)
+			(effects
+				(font
+					(size 1.27 1.27)
+				)
+			)
+		)
+		(property "Footprint" ""
+			(at 247.65 69.85 0)
+			(effects
+				(font
+					(size 1.27 1.27)
+				)
+				(hide yes)
+			)
+		)
+		(property "Datasheet" ""
+			(at 247.65 69.85 0)
+			(effects
+				(font
+					(size 1.27 1.27)
+				)
+				(hide yes)
+			)
+		)
+		(property "Description" "Power symbol creates a global label with name \"VCC\""
+			(at 247.65 69.85 0)
+			(effects
+				(font
+					(size 1.27 1.27)
+				)
+				(hide yes)
+			)
+		)
+		(pin "1"
+		)
+		(instances
+			(project "HAM_Seminar"
+				(path "/7b2739d8-9b30-4e41-8527-a1823fcf2f65"
+					(reference "#PWR015")
 					(unit 1)
 				)
@@
 		(on_board yes)
 		(dnp no)
-		(fields_autoplaced yes)
 		(property "Reference" "R8"
-			(at 220.98 91.44 90)
+			(at 219.71 77.216 90)
 			(effects
 				(font
@@
 					(size 1.27 1.27)
 				)
-			)
-		)
-		(property "Footprint" "Resistor_THT:R_Axial_DIN0204_L3.6mm_D1.6mm_P7.62mm_Horizontal"
+				(hide yes)
+			)
+		)
+		(property "Footprint" "Resistor_THT:R_Axial_DIN0207_L6.3mm_D2.5mm_P10.16mm_Horizontal"
 			(at 220.98 99.568 90)
 			(effects
@@
 		(on_board yes)
 		(dnp no)
-		(fields_autoplaced yes)
 		(property "Reference" "R9"
-			(at 220.98 93.98 90)
+			(at 219.71 79.248 90)
 			(effects
 				(font
@@
 					(size 1.27 1.27)
 				)
-			)
-		)
-		(property "Footprint" "Resistor_THT:R_Axial_DIN0204_L3.6mm_D1.6mm_P7.62mm_Horizontal"
+				(hide yes)
+			)
+		)
+		(property "Footprint" "Resistor_THT:R_Axial_DIN0207_L6.3mm_D2.5mm_P10.16mm_Horizontal"
 			(at 220.98 102.108 90)
 			(effects
@@
 			)
 		)
-		(property "Footprint" "Resistor_THT:R_Axial_DIN0204_L3.6mm_D1.6mm_P7.62mm_Horizontal"
+		(property "Footprint" "Resistor_THT:R_Axial_DIN0207_L6.3mm_D2.5mm_P10.16mm_Horizontal"
 			(at 90.932 90.17 90)
 			(effects
@@
 	)
 	(symbol
-		(lib_id "power:GND")
-		(at 247.65 114.3 0)
-		(unit 1)
-		(exclude_from_sim no)
-		(in_bom yes)
-		(on_board yes)
-		(dnp no)
-		(fields_autoplaced yes)
-		(property "Reference" "#PWR014"
-			(at 247.65 120.65 0)
-			(effects
-				(font
-					(size 1.27 1.27)
-				)
-				(hide yes)
-			)
-		)
-		(property "Value" "GND"
-			(at 247.65 119.38 0)
-			(effects
-				(font
-					(size 1.27 1.27)
-				)
-			)
-		)
-		(property "Footprint" ""
-			(at 247.65 114.3 0)
-			(effects
-				(font
-					(size 1.27 1.27)
-				)
-				(hide yes)
-			)
-		)
-		(property "Datasheet" ""
-			(at 247.65 114.3 0)
-			(effects
-				(font
-					(size 1.27 1.27)
-				)
-				(hide yes)
-			)
-		)
-		(property "Description" "Power symbol creates a global label with name \"GND\" , ground"
-			(at 247.65 114.3 0)
-			(effects
-				(font
-					(size 1.27 1.27)
-				)
-				(hide yes)
-			)
-		)
-		(pin "1"
-		)
-		(instances
-			(project "HAM_Seminar"
-				(path "/7b2739d8-9b30-4e41-8527-a1823fcf2f65"
-					(reference "#PWR014")
-					(unit 1)
-				)
-			)
-		)
-	)
-	(symbol
 		(lib_id "Device:R")
 		(at 220.98 92.71 90)
@@
 		(on_board yes)
 		(dnp no)
-		(fields_autoplaced yes)
 		(property "Reference" "R6"
-			(at 220.98 86.36 90)
+			(at 219.71 72.898 90)
 			(effects
 				(font
@@
 					(size 1.27 1.27)
 				)
-			)
-		)
-		(property "Footprint" "Resistor_THT:R_Axial_DIN0204_L3.6mm_D1.6mm_P7.62mm_Horizontal"
+				(hide yes)
+			)
+		)
+		(property "Footprint" "Resistor_THT:R_Axial_DIN0207_L6.3mm_D2.5mm_P10.16mm_Horizontal"
 			(at 220.98 94.488 90)
 			(effects
